Commit message: test

File: description/robot_core.xacro (robot description, xacro)
@@ -15,5 +15,5 @@
     </material>
     <!-- BASE LINK -->
-    <link name= "base_link">
+    <link name= "base_link_ed">
     </link>
     <!-- CHASSIS LINK -->

Commit message: Commit_2

File: description/robot_core.xacro (robot description, xacro)
@@ -15,5 +15,5 @@
     </material>
     <!-- BASE LINK -->
-    <link name= "base_link_ed">
+    <link name= "base_link">
     </link>
     <!-- CHASSIS LINK -->
